Commit message: update jh

File: src/nexus_4wd_mecanum_simulator/nexus_4wd_mecanum_description/urdf/box1.urdf (robot description, URDF)
Before this commit: robot box, 1 links, 0 joints
Links:
- link link: geometry collision cylinder length=0.4 radius=0.15; visual cylinder length=0.4 radius=0.15

File: src/nexus_4wd_mecanum_simulator/nexus_4wd_mecanum_description/urdf/box10.urdf (robot description, URDF)
Before this commit: robot box, 1 links, 0 joints
Links:
- link link: geometry collision cylinder length=0.4 radius=0.15; visual cylinder length=0.4 radius=0.15

File: src/nexus_4wd_mecanum_simulator/nexus_4wd_mecanum_description/urdf/box8.urdf (robot description, URDF)
Before this commit: robot box, 1 links, 0 joints
Links:
- link link: geometry collision cylinder length=0.4 radius=0.15; visual cylinder length=0.4 radius=0.15

File: src/nexus_4wd_mecanum_simulator/nexus_4wd_mecanum_description/urdf/test.urdf (robot description, URDF)
Before this commit: robot nexus_4wd_mecanum, 15 links, 14 joints
Links:
- link lidar_rigidbody: geometry visual cylinder length=0.2 radius=0.05
Joints:
- joint upper_lidar: origin xyz=0 0 0.001 rpy=0 0 0 -> xyz=0 0 0.1 rpy=0 0 0
